Commit message: updates

File: src/bugbot_urdf_description/urdf/bugbot_description.urdf (robot description, URDF)
Before this commit: robot serena, 4 links, 3 joints
Links:
- added link GPS
- added link IMU
- link base_link: mass 5 -> 20; geometry collision mesh filename=package://bugbot_urdf_description/meshes/BugBotBodyV3.STL; visual mesh filename=package://bugbot_urdf_description/meshes/BugBotBodyV3.STL
Joints:
- added joint GPS_joint: type fixed, parent base_link, child GPS, origin xyz=0 0 0.08223 rpy=0 0 0
- added joint IMU_joint: type fixed, parent base_link, child IMU, origin xyz=0 0 0.08223 rpy=0 0 0
- joint wheel_left_joint: origin xyz=0 0.1 0.07 rpy=1.5708 0 -3.1416 -> xyz=0 0.145 0.10223 rpy=1.5708 0 -3.1416
- joint wheel_right_joint: origin xyz=0 -0.1 0.07 rpy=1.5708 0 -3.1416 -> xyz=0 -0.145 0.10223 rpy=1.5708 0 -3.1416

Commit message: added imu and gps

File: src/bugbot_urdf_description/urdf/bugbot_description.urdf (robot description, URDF)
Before this commit: robot serena, 6 links, 5 joints
Links:
- removed link GPS
- added link GPS_link
Joints:
- joint GPS_joint: child GPS -> GPS_link

Commit message: friction adjustment

File: src/bugbot_urdf_description/urdf/bugbot_description.urdf (robot description, URDF)
Before this commit: robot serena, 6 links, 5 joints
Links:
- link base_link: mass 20 -> 5
